File: BabysFirstCell.kicad_sch (KiCad schematic)
At the start: 18 parts, among them J1 Uart vcc gnd rx tx, J2 Head, J3 Conn_01x05, U2 MCP1703Ax-330xxTT, U3 STM32G051F8Px

Commit message: Add EasyEDA Pro project files
Parts:
- C6: footprint Capacitor_SMD:C_01005_0402Metric -> Resistor_SMD:R_0603_1608Metric
- J2: footprint Connector_Molex:Molex_KK-254_AE-6410-04A_1x04_P2.54mm_Vertical -> Connector_JST:JST_PH_B4B-PH-K_1x04_P2.00mm_Vertical
Connections:
- no-connect marks 12 -> 14
Changed lines of the file:
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@@
+	)
+	(junction
+		(at 109.22 52.07)
+		(diameter 0)
+		(color 0 0 0 0)
+	)
+	(junction
+		(at 120.65 72.39)
+		(diameter 0)
+		(color 0 0 0 0)
+	)
+	(junction
+		(at 80.01 52.07)
+		(diameter 0)
+		(color 0 0 0 0)
+	)
+	(junction
+		(at 146.05 64.77)
+		(diameter 0)
+		(color 0 0 0 0)
+	)
+	(junction
+		(at 189.23 68.58)
+		(diameter 0)
+		(color 0 0 0 0)
+	)
+	(junction
+		(at 207.01 55.88)
+		(diameter 0)
+		(color 0 0 0 0)
+	)
+	(junction
+		(at 139.7 55.88)
+		(diameter 0)
+		(color 0 0 0 0)
+	)
+	(junction
+		(at 86.36 57.15)
+		(diameter 0)
+		(color 0 0 0 0)
+	)
+	(junction
+		(at 182.88 55.88)
+		(diameter 0)
+		(color 0 0 0 0)
 	)
 	(junction
@@
 	)
 	(junction
-		(at 109.22 52.07)
-		(diameter 0)
-		(color 0 0 0 0)
-	)
-	(junction
-		(at 120.65 72.39)
-		(diameter 0)
-		(color 0 0 0 0)
-	)
-	(junction
-		(at 80.01 52.07)
-		(diameter 0)
-		(color 0 0 0 0)
-	)
-	(junction
-		(at 146.05 64.77)
-		(diameter 0)
-		(color 0 0 0 0)
-	)
-	(junction
-		(at 189.23 68.58)
-		(diameter 0)
-		(color 0 0 0 0)
-	)
-	(junction
-		(at 207.01 55.88)
-		(diameter 0)
-		(color 0 0 0 0)
-	)
-	(junction
-		(at 139.7 55.88)
-		(diameter 0)
-		(color 0 0 0 0)
-	)
-	(junction
-		(at 86.36 57.15)
-		(diameter 0)
-		(color 0 0 0 0)
-	)
-	(junction
-		(at 182.88 55.88)
-		(diameter 0)
-		(color 0 0 0 0)
-	)
-	(junction
 		(at 102.87 60.96)
 		(diameter 0)
@@
 	)
 	(no_connect
+		(at 187.96 48.26)
+	)
+	(no_connect
 		(at 184.15 87.63)
 	)
@@
 	)
 	(no_connect
+		(at 217.17 49.53)
+	)
+	(no_connect
 		(at 184.15 92.71)
 	)
@@
 	(wire
 		(pts
+			(xy 146.05 64.77) (xy 153.67 64.77)
+		)
+		(stroke
+			(width 0)
+			(type default)
+		)
+	)
+	(wire
+		(pts
 			(xy 87.63 52.07) (xy 86.36 52.07)
 		)
@@
 	(wire
 		(pts
-			(xy 146.05 64.77) (xy 153.67 64.77)
-		)
-		(stroke
-			(width 0)
-			(type default)
-		)
-	)
-	(wire
-		(pts
 			(xy 177.8 53.34) (xy 177.8 55.88)
 		)
@@
 	(wire
 		(pts
+			(xy 153.67 49.53) (xy 153.67 64.77)
+		)
+		(stroke
+			(width 0)
+			(type default)
+		)
+	)
+	(wire
+		(pts
 			(xy 139.7 55.88) (xy 146.05 55.88)
 		)
@@
 	(wire
 		(pts
-			(xy 153.67 64.77) (xy 153.67 66.04)
-		)
-		(stroke
-			(width 0)
-			(type default)
-		)
-	)
-	(wire
-		(pts
 			(xy 182.88 53.34) (xy 182.88 55.88)
 		)
@@
 		(pts
 			(xy 86.36 57.15) (xy 86.36 60.96)
-		)
-		(stroke
-			(width 0)
-			(type default)
-		)
-	)
-	(wire
-		(pts
-			(xy 153.67 49.53) (xy 153.67 64.77)
 		)
 		(stroke
@@
 			)
 		)
-		(property "Footprint" "Connector_Molex:Molex_KK-254_AE-6410-04A_1x04_P2.54mm_Vertical"
+		(property "Footprint" "Connector_JST:JST_PH_B4B-PH-K_1x04_P2.00mm_Vertical"
 			(at 177.8 48.26 0)
 			(hide yes)
@@
 			)
 		)
-		(property "Footprint" "Capacitor_SMD:C_01005_0402Metric"
+		(property "Footprint" "Resistor_SMD:R_0603_1608Metric"
 			(at 80.01 54.61 0)
 			(hide yes)
